File: hardware/malt/malt.kicad_pcb (KiCad board)
At the start: 2 copper layers, 99.7 x 64.1 mm, 33 parts, among them CN1 MSX_SLOT_CON, P40 PINHD-02x20, P44 Conn_02x22, T1 TestPoint, T12 TestPoint, T2 TestPoint, T3 TestPoint, T42 TestPoint, T49 TestPoint, T6 TestPoint, T7 TestPoint, T8 TestPoint, T9 TestPoint, U1 SST39SF0X0, U2 82C55A, U3 74HCT32, U4 74HCT04, U5 74HCT138

Commit message: malt v1.2
see issue #16
Parts:
- added R5: 10K, Resistor_THT:R_Axial_DIN0204_L3.6mm_D1.6mm_P7.62mm_Horizontal, F.Cu at (107.6, 63.5)
- added SW1: PIN_1x3, Button_Switch_THT:SW_Slide_SPDT_Angled_CK_OS102011MA1Q, F.Cu at (188.6, 59.2)
- moved C1 1.97 mm to (188.6, 104.0)
- moved JP3 1.44 mm to (101.2, 69.4)
- moved U1 1.38 mm to (194.2, 100.1)
- moved U5 0.28 mm to (107.6, 91.3)
- moved R1 0.13 mm to (118.9, 63.5)
- moved C4 0.13 mm to (112.6, 85.2)
- renumbered JP4 to JP3, JP3 to SW2
Connections:
- net Net-(JP1-C) renamed /A16
- SW2 pad 1: VCC -> Net-(SW2-A)
- SW2 pad 2: Net-(JP3-C) -> Net-(SW2-C)
- SW2 pad 3: /~{RD} -> GND
- U1 pad 22: /~{SLTSL} -> /~{ROMCE}
- U1 pad 24: Net-(JP3-C) -> /~{RD}
- U3 pad 10: Net-(U3-Pad10) -> /~{SLTSL}
- U3 pad 11: Net-(U3-Pad10) -> unconnected-(U3-Pad11)
- U3 pad 8: unconnected-(U3-Pad8) -> /~{ROMCE}
- U3 pad 9: Net-(U3-Pad10) -> Net-(SW2-C)
Routing:
- net /~{ROMCE}: track 0.00 -> 112.6 mm
- net Net-(JP3-C): track 98.8 -> 0.00 mm
- net /~{HCS1}: track 17.4 -> 59.4 mm
- net /A8: track 91.6 -> 53.7 mm, vias 4 -> 2
- net VCC: track 242.3 -> 278.0 mm, vias 0 -> 1
- net Net-(SW2-C): track 0.00 -> 35.1 mm
- net /~{SLTSL}: track 59.7 -> 93.7 mm, vias 2 -> 3
- net /~{RD}: track 138.7 -> 105.5 mm
- net /A2: track 186.5 -> 158.2 mm, vias 4 -> 3
- net GND: track 373.9 -> 395.9 mm, vias 1 -> 2
- net /A16: track 44.6 -> 59.7 mm, vias 2 -> 3
- net /D5: track 108.9 -> 96.5 mm, vias 4 -> 2
- net /A6: track 144.7 -> 154.6 mm
- net /A4: track 128.6 -> 136.2 mm, vias 2 -> 3
- net Net-(SW2-A): track 0.00 -> 7.37 mm
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Other:
- board text added: "MALT IDE V1.2"
- board text removed: "MALT IDE V1.1"
