File: hardware/malt/malt.kicad_sch (KiCad schematic)
At the start: 33 parts, among them CN1 MSX_SLOT_CON, P40 PINHD-02x20, P44 Conn_02x22, T1 TestPoint, T12 TestPoint, T2 TestPoint, T3 TestPoint, T42 TestPoint, T49 TestPoint, T6 TestPoint, T7 TestPoint, T8 TestPoint, T9 TestPoint, U1 SST39SF0X0, U2 82C55A, U3 74HCT32, U4 74HCT04, U5 74HCT138

Commit message: malt v1.2
see issue #16
Parts:
- added R5: 10K, Resistor_THT:R_Axial_DIN0204_L3.6mm_D1.6mm_P7.62mm_Horizontal, symbol Device:R
- added SW1: PIN_1x3, Button_Switch_THT:SW_Slide_SPDT_Angled_CK_OS102011MA1Q, symbol Jumper:Jumper_3_Bridged12
- renumbered JP4 to JP3, JP3 to SW2
Connections:
- net GND: now also SW2.3 (B), SW1.3 (B)
- net VCC: now also R5.1, SW1.1 (A); no longer SW2.1 (A)
- net ~{RD}: now also U1.24 (OE); no longer SW2.3 (B)
- net ~{SLTSL}: now also U3.10; no longer U1.22 (CE)
- net ~{ROMCE}: now reaches U3.8
- net ~{ROMCE}: now also U1.22 (CE)
- net A16: now reaches JP1.2 (C), U1.2 (A16)
- net A16: now also SW1.2 (C)
- net at SW2.2 (C): now also U3.9; no longer U1.24 (OE)
- new net: R5.2, SW2.1 (A)
- now unconnected: U3.11
Other:
- note added: "Alternative bank switch"
- note added: "Disable ROM Enable"
- note added: "U1 options: SST39SF010A SST39SF020A SST39SF040 W27C512 (no switch)"
- note removed: "U1 options: SST39SF010A SST39SF020A SST39SF040A W27C512 (NO JP1)"
- moved on the sheet: C1, C2, C3, C4, C5, C6, SW2, U3C, U3D, U3E, U4G
